Commit message: feat: 增加 usb_cdc intent 调试覆盖并更新机器人与任务配置
  - 为 usb_cdc_node 增加 intent 调试覆盖参数和动态回调
  - 增加 tx 安全门控与启动关节目标写入
  - 将夹爪协议切换为开合命令
  - 补充执行与规划调试日志，调整任务超时与轨迹配置
  - 更新机器人 URDF、手指模型、碰撞矩阵与 MoveIt 配置
  - 增加 pose_marker_node 资源与文档

File: src/robots/engineer_description/urdf/engineer_v5.urdf (robot description, URDF)
Before this commit: robot engineer_description, 10 links, 9 joints
Links:
- link camera_link: mass 0.10407354521816 -> 0.104061987455649; geometry collision mesh filename=package://engineer_description/dae/camera_link.dae; visual mesh filename=package://engineer_description/dae/camera_link.dae
- link left_gripper_link: mass 0.0642787256124548 -> 0.0642787256124547; geometry collision mesh filename=package://engineer_description/dae_collision/left_finger_li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; visual mesh filename=package://engineer_description/dae/left_finger_link.dae
- link link1: mass 1.17124495128858 -> 1.21588615841954
- link link2: mass 0.962417455746602 -> 0.971751552734983
- link link3: mass 0.614016140789944 -> 0.63413356071165
- link link4: mass 0.407781795652674 -> 0.407781795652687
- link link6: mass 0.286453096129479 -> 0.286453096129476
- link right_gripper_link: mass 0.0642787256124545 -> 0.0642787256124544; geometry collision mesh filename=package://engineer_description/dae_collision/right_finger_l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; visual mesh filename=package://engineer_description/dae/right_finger_link.dae
Joints:
- joint camera_joint: origin xyz=-0.0349999999999999 0.0849279748513231 0.0615000049599689 rpy=-1.5707963267949 0 0 -> xyz=-0.0349999999999999 -0.0189726950499375 0.0614999950400312 rpy=-1.5707963267949 0 1.5707963267949
- joint joint1: origin xyz=0.086 0 0.035001 rpy=0 0 0 -> xyz=0.0859996586366104 0 0.0350008387668869 rpy=0 0 0
- joint joint2: limit lower=-3.14 upper=3.14 effort=0 velocity=0 -> lower=-1.2399 upper=1.1779 effort=0 velocity=0; origin xyz=0 0 0.119 rpy=1.5708 0 0 -> xyz=0 0 0.119 rpy=-1.57079632679489 -1.48352986419519 3.14159265358979
- joint joint3: limit lower=-3.14 upper=3.14 effort=0 velocity=0 -> lower=-2.7113 upper=2.4329 effort=0 velocity=0; origin xyz=0 0.390000000000001 0.0192 rpy=0 0 0 -> xyz=0.388515932255782 -0.033990739671585 0.0192000000000002 rpy=0 0 -1.65806278939461
- joint joint4: origin xyz=0 0.114 0.039 rpy=-1.5708 0 0 -> xyz=0 0.114000000000009 0.0390000000000176 rpy=-1.5707963267949 0 0
- joint joint5: limit lower=-3.14 upper=3.14 effort=0 velocity=0 -> lower=-1.85 upper=1.85 effort=0 velocity=0; origin xyz=0 0 0.23 rpy=1.5708 0 0 -> xyz=0 0 0.229999999999999 rpy=1.5707963267949 0 0
- joint joint6: origin xyz=0 0.007 0 rpy=1.5708 1.5708 0 -> xyz=0 0.00700000000000101 0 rpy=1.5707963267949 1.5707963267949 0
- joint right_gripper_joint: mimic joint=left_gripper_joint multiplier=1 offset=0 -> joint=left_gripper_joint multiplier=-1 offset=0
